Commit message: new movit_config package witsh working execution, fixed errors in ros2_controller and movit_controller. next to do setup gripper controller attached to gripper end effector

File: mycobot_movit_config/config/mycobot_280.ros2_control.xacro (robot description, xacro)
@@ -38,4 +38,10 @@
                 </state_interface>
             </joint>
+            <joint name="link6_to_link6flange">
+                <command_interface name="position"/>
+                <state_interface name="position">
+                  <param name="initial_value">${initial_positions['link6_to_link6flange']}</param>
+                </state_interface>
+            </joint>
         </ros2_control>
     </xacro:macro>

Commit message: gripper action added but currently not working, arm execution is fine

File: mycobot_movit_config/config/mycobot_280.ros2_control.xacro (robot description, xacro)
@@ -44,4 +44,10 @@
                 </state_interface>
             </joint>
+            <joint name="gripper_controller">
+                <command_interface name="position"/>
+                <state_interface name="position">
+                  <param name="initial_value">${initial_positions['gripper_controller']}</param>
+                </state_interface>
+            </joint>
         </ros2_control>
     </xacro:macro>
