Commit message: configure cobot in gazebo world attempt, though full of errors this can still be used as a reference point, will be reverting back to follow docs procedure or video tutorial

File: ros-packages/mycobot_description/urdf/mycobot_280_urdf.xacro (robot description, xacro)
@@ -504,3 +504,85 @@
 		<mimic joint="gripper_controller" multiplier="1.0" offset="0" />
 	</joint>
+<!-- ********** TRANSMISSIONS ********** -->
+	<!-- Only revolute joints need transmissions. Fixed joints do not. -->
+	<!-- Arm Joint Transmissions -->
+	<transmission name="link1_to_link2_trans">
+		<type>transmission_interface/SimpleTransmission</type>
+		<joint name="link1_to_link2">
+			<hardwareInterface>hardware_interface/PositionJointInterface</hardwareInterface>
+		</joint>
+		<actuator name="link1_to_link2_motor">
+			<mechanicalReduction>1</mechanicalReduction>
+			<hardwareInterface>hardware_interface/PositionJointInterface</hardwareInterface>
+		</actuator>
+	</transmission>
+	<transmission name="link2_to_link3_trans">
+		<type>transmission_interface/SimpleTransmission</type>
+		<joint name="link2_to_link3">
+			<hardwareInterface>hardware_interface/PositionJointInterface</hardwareInterface>
+		</joint>
+		<actuator name="link2_to_link3_motor">
+			<mechanicalReduction>1</mechanicalReduction>
+			<hardwareInterface>hardware_interface/PositionJointInterface</hardwareInterface>
+		</actuator>
+	</transmission>
+	<transmission name="link3_to_link4_trans">
+		<type>transmission_interface/SimpleTransmission</type>
+		<joint name="link3_to_link4">
+			<hardwareInterface>hardware_interface/PositionJointInterface</hardwareInterface>
+		</joint>
+		<actuator name="link3_to_link4_motor">
+			<mechanicalReduction>1</mechanicalReduction>
+			<hardwareInterface>hardware_interface/PositionJointInterface</hardwareInterface>
+		</actuator>
+	</transmission>
+	<transmission name="link4_to_link5_trans">
+		<type>transmission_interface/SimpleTransmission</type>
+		<joint name="link4_to_link5">
+			<hardwareInterface>hardware_interface/PositionJointInterface</hardwareInterface>
+		</joint>
+		<actuator name="link4_to_link5_motor">
+			<mechanicalReduction>1</mechanicalReduction>
+			<hardwareInterface>hardware_interface/PositionJointInterface</hardwareInterface>
+		</actuator>
+	</transmission>
+	<transmission name="link5_to_link6_trans">
+		<type>transmission_interface/SimpleTransmission</type>
+		<joint name="link5_to_link6">
+			<hardwareInterface>hardware_interface/PositionJointInterface</hardwareInterface>
+		</joint>
+		<actuator name="link5_to_link6_motor">
+			<mechanicalReduction>1</mechanicalReduction>
+			<hardwareInterface>hardware_interface/PositionJointInterface</hardwareInterface>
+		</actuator>
+	</transmission>
+	<transmission name="link6_to_link6flange_trans">
+		<type>transmission_interface/SimpleTransmission</type>
+		<joint name="link6_to_link6flange">
+			<hardwareInterface>hardware_interface/PositionJointInterface</hardwareInterface>
+		</joint>
+		<actuator name="link6_to_link6flange_motor">
+			<mechanicalReduction>1</mechanicalReduction>
+			<hardwareInterface>hardware_interface/PositionJointInterface</hardwareInterface>
+		</actuator>
+	</transmission>
+	<!-- Gripper Joint Transmission -->
+<transmission name="gripper_controller_trans">
+  <type>transmission_interface/SimpleTransmission</type>
+  <joint name="gripper_controller">
+    <hardwareInterface>hardware_interface/PositionJointInterface</hardwareInterface>
+  </joint>
+  <actuator name="gripper_motor">
+    <mechanicalReduction>1</mechanicalReduction>
+    <hardwareInterface>hardware_interface/PositionJointInterface</hardwareInterface>
+  </actuator>
+</transmission>
+	<!--gazebo plugin -->
+<gazebo>
+  <plugin name="gazebo_ros2_control" filename="libgazebo_ros2_control.so">
+    <robotNamespace>/robot_arm</robotNamespace>
+    <robotSimType>gazebo_ros2_control/GazeboSystem</robotSimType>
+    <parametersFile>$(mycobot_movit_config)/config/ros2_controllers.yaml</parametersFile>
+  </plugin>
+</gazebo>
 </robot>

Commit message: undid broken gazebo setup will use official guidelines for next attempt

File: ros-packages/mycobot_description/urdf/mycobot_280_urdf.xacro (robot description, xacro)
@@ -504,85 +504,3 @@
 		<mimic joint="gripper_controller" multiplier="1.0" offset="0" />
 	</joint>
-<!-- ********** TRANSMISSIONS ********** -->
-	<!-- Only revolute joints need transmissions. Fixed joints do not. -->
-	<!-- Arm Joint Transmissions -->
-	<transmission name="link1_to_link2_trans">
-		<type>transmission_interface/SimpleTransmission</type>
-		<joint name="link1_to_link2">
-			<hardwareInterface>hardware_interface/PositionJointInterface</hardwareInterface>
-		</joint>
-		<actuator name="link1_to_link2_motor">
-			<mechanicalReduction>1</mechanicalReduction>
-			<hardwareInterface>hardware_interface/PositionJointInterface</hardwareInterface>
-		</actuator>
-	</transmission>
-	<transmission name="link2_to_link3_trans">
-		<type>transmission_interface/SimpleTransmission</type>
-		<joint name="link2_to_link3">
-			<hardwareInterface>hardware_interface/PositionJointInterface</hardwareInterface>
-		</joint>
-		<actuator name="link2_to_link3_motor">
-			<mechanicalReduction>1</mechanicalReduction>
-			<hardwareInterface>hardware_interface/PositionJointInterface</hardwareInterface>
-		</actuator>
-	</transmission>
-	<transmission name="link3_to_link4_trans">
-		<type>transmission_interface/SimpleTransmission</type>
-		<joint name="link3_to_link4">
-			<hardwareInterface>hardware_interface/PositionJointInterface</hardwareInterface>
-		</joint>
-		<actuator name="link3_to_link4_motor">
-			<mechanicalReduction>1</mechanicalReduction>
-			<hardwareInterface>hardware_interface/PositionJointInterface</hardwareInterface>
-		</actuator>
-	</transmission>
-	<transmission name="link4_to_link5_trans">
-		<type>transmission_interface/SimpleTransmission</type>
-		<joint name="link4_to_link5">
-			<hardwareInterface>hardware_interface/PositionJointInterface</hardwareInterface>
-		</joint>
-		<actuator name="link4_to_link5_motor">
-			<mechanicalReduction>1</mechanicalReduction>
-			<hardwareInterface>hardware_interface/PositionJointInterface</hardwareInterface>
-		</actuator>
-	</transmission>
-	<transmission name="link5_to_link6_trans">
-		<type>transmission_interface/SimpleTransmission</type>
-		<joint name="link5_to_link6">
-			<hardwareInterface>hardware_interface/PositionJointInterface</hardwareInterface>
-		</joint>
-		<actuator name="link5_to_link6_motor">
-			<mechanicalReduction>1</mechanicalReduction>
-			<hardwareInterface>hardware_interface/PositionJointInterface</hardwareInterface>
-		</actuator>
-	</transmission>
-	<transmission name="link6_to_link6flange_trans">
-		<type>transmission_interface/SimpleTransmission</type>
-		<joint name="link6_to_link6flange">
-			<hardwareInterface>hardware_interface/PositionJointInterface</hardwareInterface>
-		</joint>
-		<actuator name="link6_to_link6flange_motor">
-			<mechanicalReduction>1</mechanicalReduction>
-			<hardwareInterface>hardware_interface/PositionJointInterface</hardwareInterface>
-		</actuator>
-	</transmission>
-	<!-- Gripper Joint Transmission -->
-<transmission name="gripper_controller_trans">
-  <type>transmission_interface/SimpleTransmission</type>
-  <joint name="gripper_controller">
-    <hardwareInterface>hardware_interface/PositionJointInterface</hardwareInterface>
-  </joint>
-  <actuator name="gripper_motor">
-    <mechanicalReduction>1</mechanicalReduction>
-    <hardwareInterface>hardware_interface/PositionJointInterface</hardwareInterface>
-  </actuator>
-</transmission>
-	<!--gazebo plugin -->
-<gazebo>
-  <plugin name="gazebo_ros2_control" filename="libgazebo_ros2_control.so">
-    <robotNamespace>/robot_arm</robotNamespace>
-    <robotSimType>gazebo_ros2_control/GazeboSystem</robotSimType>
-    <parametersFile>$(mycobot_movit_config)/config/ros2_controllers.yaml</parametersFile>
-  </plugin>
-</gazebo>
 </robot>
